File: PCB/time-o-matic/time-o-matic.kicad_sch (KiCad schematic)
At the start: 30 parts, among them J1 Conn_01x02_Pin, J2 USB_C_Receptacle_USB2.0_14P, U1 ESP32-WROOM-E, U2 MP1584EN-LF-P, U3 TP4056-42-ESOP8, U4 CH340C

Commit message: Updating Schematic
Parts:
- removed C5, C6: 10uF, symbol Device:C
- removed D2, D3: LED, symbol Device:LED
- removed R7, R8: 1k, symbol Device:R
- removed U3: TP4056-42-ESOP8, Package_SO:SOIC-8-1EP_3.9x4.9mm_P1.27mm_EP2.41x3.3mm_ThermalVias, symbol Battery_Management:TP4056-42-ESOP8
- added J3: Power TP4056, symbol Connector:Conn_01x02_Pin
- added J4: GPS connector, symbol Connector:Conn_01x04_Socket
- added SW1, SW2, SW3, SW4, SW5, SW6: SW_Push, symbol Switch:SW_Push
- J1: value Conn_01x02_Pin -> Power from Battery
Connections:
- net +3V3: now also J4.1 (Pin_1)
- net +5V: now also J3.2 (Pin_2)
- net Earth: no longer C1.2, C3.2, D1.1 (K), J1.1 (Pin_1), J2.A1 (GND), J2.A12 (GND), J2.B1 (GND), J2.B12 (GND), J2.S1 (SHIELD), R10.1, R2.1, R3.1, R4.1, R6.1, R9.1, U1.1 (GND), U1.15 (GND), U1.38 (GND), U1.39 (GND_THERMAL), U2.5 (GND)
- net VIN: now also J1.1 (Pin_1)
- net GND: now reaches J1.2 (Pin_2)
- net GND: now also C1.2, C3.2, D1.1 (K), J2.A1 (GND), J2.A12 (GND), J2.B1 (GND), J2.B12 (GND), J2.S1 (SHIELD), R10.1, R2.1, R3.1, R4.1, R6.1, R9.1, U1.1 (GND), U1.15 (GND), U1.38 (GND), U1.39 (GND_THERMAL), U2.5 (GND), J3.1 (Pin_1), J4.4 (Pin_4), SW1.1, SW2.1, SW3.1, SW4.1, SW5.1, SW6.1
- net RX: now reaches U1.11 (DAC_2/ADC2_CH9/GPIO26)
- net RX: now also J4.3 (Pin_3)
- net TX: now reaches U1.12 (ADC2_CH7/GPIO27)
- net TX: now also J4.2 (Pin_2)
- net SW1: now reaches U1.27 (GPIO16)
- net SW1: now also SW1.2
- net SW2: now reaches U1.28 (GPIO17)
- net SW2: now also SW2.2
- net SW3: now reaches U1.30 (GPIO18)
- net SW3: now also SW3.2
- net SW4: now reaches U1.31 (GPIO19)
- net SW4: now also SW4.2
- net SW5: now reaches U1.33 (GPIO21)
- net SW5: now also SW5.2
- net SW6: now reaches U1.36 (GPIO22)
- net SW6: now also SW6.2
Other:
- note added: "I/O"
- note added: "MCU ESP32"
- note added: "Power Input + UART Converter"
- note added: "Voltage Regulator"
- moved on the sheet: C1, C2, C3, C4, C7, C8, D1, J2, L1, R1, R10, R11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

Commit message: W
Parts:
- removed J1: Power from Battery, symbol Connector:Conn_01x02_Pin
- removed J3: Power TP4056, symbol Connector:Conn_01x02_Pin
- removed J4: GPS connector, symbol Connector:Conn_01x04_Socket
- removed SW1, SW2, SW3, SW4, SW5, SW6: SW_Push, symbol Switch:SW_Push
- added J5: Display Connector, Connector_PinHeader_2.54mm:PinHeader_1x04_P2.54mm_Vertical, symbol Connector:Conn_01x04_Socket
- C1, C2, C3, C4, C7, C8: footprint (none) -> Capacitor_SMD:C_0603_1608Metric_Pad1.08x0.95mm_HandSolder
- D1: footprint (none) -> Diode_SMD:D_3220_8050Metric_Pad2.65x5.15mm_HandSolder
- J2: footprint (none) -> Connector_USB:USB_C_Receptacle_GCT_USB4085
- L1: footprint (none) -> Inductor_SMD:L_0603_1608Metric_Pad1.05x0.95mm_HandSolder
- R1, R10, R11, R12, R2, R3, R4, R5, R6, R9: footprint (none) -> Resistor_SMD:R_0603_1608Metric_Pad0.98x0.95mm_HandSolder
Connections:
- net +5V is gone; now on net VIN: J2.A4 (VBUS), J2.A9 (VBUS), J2.B4 (VBUS), J2.B9 (VBUS)
- net Earth is gone; now on net GND: C7.2, C8.1, U4.1 (GND)
- net +3V3: now also J5.1 (Pin_1)
- net GND: now also J5.4 (Pin_4)
- net i2c-: now reaches U1.10 (DAC_1/ADC2_CH8/GPIO25)
- net i2c-: now also J5.3 (Pin_3)
- net i2c+: now reaches U1.7 (GPIO35/ADC1_CH7)
- net i2c+: now also J5.2 (Pin_2)
- net RX: no longer names the net of U1.11 (DAC_2/ADC2_CH9/GPIO26)
- net RXD renamed P
- net SW1: no longer names the net of U1.27 (GPIO16)
- net SW2: no longer names the net of U1.28 (GPIO17)
- net SW3: no longer names the net of U1.30 (GPIO18)
- net SW4: no longer names the net of U1.31 (GPIO19)
- net SW5: no longer names the net of U1.33 (GPIO21)
- net SW6: no longer names the net of U1.36 (GPIO22)
- net TX: no longer names the net of U1.12 (ADC2_CH7/GPIO27)
- net TXD renamed N
Other:
- note added: "MCU ESP32 WROOM"
- note removed: "MCU ESP32"
- moved on the sheet: C1, C2, C3, C4, C7, C8, D1, J2, L1, R1, R10, R11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
