File: PCB/time-o-matic.kicad_pcb (KiCad board)
At the start: 2 copper layers, 60.8 x 74.1 mm, 23 parts, among them J2 USB_C_Receptacle_USB2.0_14P, J5 Display Connector, U1 ESP32-WROOM-E, U2 MP1584EN-LF-P, U4 CH340C

Commit message: W
Parts:
- D1: footprint Diode_SMD:D_3220_8050Metric_Pad2.65x5.15mm_HandSolder -> Diode_SMD:D_SOD-882
- moved D1 5.35 mm to (118.9, 96.4)
Routing:
- net SW: track 54.1 -> 49.9 mm
Changed lines of the file:
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@@
 		)
 	)
-	(footprint "Diode_SMD:D_3220_8050Metric_Pad2.65x5.15mm_HandSolder"
-		(layer "F.Cu")
-		(at 123.42 93.46 -90)
-		(descr "Diode SMD 3220 (8050 Metric), square (rectangular) end terminal, IPC_7351 nominal, (Body size from: http://datasheets.avx.com/schottky.pdf), generated with kicad-footprint-generator")
-		(tags "diode handsolder")
+	(footprint "Diode_SMD:D_SOD-882"
+		(layer "F.Cu")
+		(at 118.93 96.3725 -90)
+		(descr "SOD-882, DFN1006-2, body 1.0 x 0.6 x 0.48mm, pitch 0.65mm, https://assets.nexperia.com/documents/package-information/SOD882.pdf")
+		(tags "Diode SOD882 DFN1006-2")
 		(property "Reference" "D1"
-			(at 0 -3.52 90)
+			(at 0 -1.35 270)
 			(layer "F.SilkS")
 			(effects
@@
 		)
 		(property "Value" "D_Schottky"
-			(at 0 3.52 90)
+			(at 0 1.35 270)
 			(layer "F.Fab")
 			(effects
@@
 		(attr smd)
 		(fp_line
-			(start -4.86 2.835)
-			(end 4 2.835)
-			(stroke
-				(width 0.12)
-				(type solid)
-			)
-			(layer "F.SilkS")
-		)
-		(fp_line
-			(start -4.86 -2.835)
-			(end -4.86 2.835)
-			(stroke
-				(width 0.12)
-				(type solid)
-			)
-			(layer "F.SilkS")
-		)
-		(fp_line
-			(start 4 -2.835)
-			(end -4.86 -2.835)
-			(stroke
-				(width 0.12)
-				(type solid)
-			)
-			(layer "F.SilkS")
-		)
-		(fp_line
-			(start -4.85 2.82)
-			(end -4.85 -2.82)
-			(stroke
-				(width 0.05)
-				(type solid)
-			)
-			(layer "F.CrtYd")
-		)
-		(fp_line
-			(start 4.85 2.82)
-			(end -4.85 2.82)
-			(stroke
-				(width 0.05)
-				(type solid)
-			)
-			(layer "F.CrtYd")
-		)
-		(fp_line
-			(start -4.85 -2.82)
-			(end 4.85 -2.82)
-			(stroke
-				(width 0.05)
-				(type solid)
-			)
-			(layer "F.CrtYd")
-		)
-		(fp_line
-			(start 4.85 -2.82)
-			(end 4.85 2.82)
-			(stroke
-				(width 0.05)
-				(type solid)
-			)
-			(layer "F.CrtYd")
-		)
-		(fp_line
-			(start -4 2.5)
-			(end 4 2.5)
-			(stroke
-				(width 0.1)
-				(type solid)
-			)
-			(layer "F.Fab")
-		)
-		(fp_line
-			(start 4 2.5)
-			(end 4 -2.5)
-			(stroke
-				(width 0.1)
-				(type solid)
-			)
-			(layer "F.Fab")
-		)
-		(fp_line
-			(start -4 -1.5)
-			(end -4 2.5)
-			(stroke
-				(width 0.1)
-				(type solid)
-			)
-			(layer "F.Fab")
-		)
-		(fp_line
-			(start -3 -2.5)
-			(end -4 -1.5)
-			(stroke
-				(width 0.1)
-				(type solid)
-			)
-			(layer "F.Fab")
-		)
-		(fp_line
-			(start 4 -2.5)
-			(end -3 -2.5)
+			(start -0.81 0.61)
+			(end 0.5 0.61)
+			(stroke
+				(width 0.12)
+				(type solid)
+			)
+			(layer "F.SilkS")
+		)
+		(fp_line
+			(start -0.81 -0.61)
+			(end -0.81 0.61)
+			(stroke
+				(width 0.12)
+				(type solid)
+			)
+			(layer "F.SilkS")
+		)
+		(fp_line
+			(start -0.81 -0.61)
+			(end 0.5 -0.61)
+			(stroke
+				(width 0.12)
+				(type solid)
+			)
+			(layer "F.SilkS")
+		)
+		(fp_line
+			(start 0.8 0.6)
+			(end -0.8 0.6)
+			(stroke
+				(width 0.05)
+				(type solid)
+			)
+			(layer "F.CrtYd")
+		)
+		(fp_line
+			(start -0.8 -0.6)
+			(end -0.8 0.6)
+			(stroke
+				(width 0.05)
+				(type solid)
+			)
+			(layer "F.CrtYd")
+		)
+		(fp_line
+			(start -0.8 -0.6)
+			(end 0.8 -0.6)
+			(stroke
+				(width 0.05)
+				(type solid)
+			)
+			(layer "F.CrtYd")
+		)
+		(fp_line
+			(start 0.8 -0.6)
+			(end 0.8 0.6)
+			(stroke
+				(width 0.05)
+				(type solid)
+			)
+			(layer "F.CrtYd")
+		)
+		(fp_line
+			(start -0.5 0.3)
+			(end -0.5 -0.3)
+			(stroke
+				(width 0.1)
+				(type solid)
+			)
+			(layer "F.Fab")
+		)
+		(fp_line
+			(start 0.5 0.3)
+			(end -0.5 0.3)
+			(stroke
+				(width 0.1)
+				(type solid)
+			)
+			(layer "F.Fab")
+		)
+		(fp_line
+			(start -0.15 0.2)
+			(end -0.15 -0.2)
+			(stroke
+				(width 0.1)
+				(type solid)
+			)
+			(layer "F.Fab")
+		)
+		(fp_line
+			(start 0.15 0.2)
+			(end 0.15 -0.2)
+			(stroke
+				(width 0.1)
+				(type solid)
+			)
+			(layer "F.Fab")
+		)
+		(fp_line
+			(start -0.15 0)
+			(end 0.15 0.2)
+			(stroke
+				(width 0.1)
+				(type solid)
+			)
+			(layer "F.Fab")
+		)
+		(fp_line
+			(start -0.15 0)
+			(end -0.3 0)
+			(stroke
+				(width 0.1)
+				(type solid)
+			)
+			(layer "F.Fab")
+		)
+		(fp_line
+			(start 0.15 0)
+			(end 0.3 0)
+			(stroke
+				(width 0.1)
+				(type solid)
+			)
+			(layer "F.Fab")
+		)
+		(fp_line
+			(start 0.15 -0.2)
+			(end -0.15 0)
+			(stroke
+				(width 0.1)
+				(type solid)
+			)
+			(layer "F.Fab")
+		)
+		(fp_line
+			(start -0.5 -0.3)
+			(end 0.5 -0.3)
+			(stroke
+				(width 0.1)
+				(type solid)
+			)
+			(layer "F.Fab")
+		)
+		(fp_line
+			(start 0.5 -0.3)
+			(end 0.5 0.3)
 			(stroke
 				(width 0.1)
@@
 		)
 		(fp_text user "${REFERENCE}"
-			(at 0 0 90)
+			(at -0.127 -1.35 270)
 			(layer "F.Fab")
 			(effects
@@
 			)
 		)
+		(pad "" smd roundrect
+			(at -0.35 0 270)
+			(size 0.3 0.6)
+			(layers "F.Paste")
+			(roundrect_rratio 0.1666666667)
+			(solder_paste_margin -0.05)
+		)
+		(pad "" smd roundrect
+			(at 0.35 0 270)
+			(size 0.3 0.6)
+			(layers "F.Paste")
+			(roundrect_rratio 0.1666666667)
+			(solder_paste_margin -0.05)
+		)
 		(pad "1" smd roundrect
-			(at -3.275 0 270)
-			(size 2.65 5.15)
-			(layers "F.Cu" "F.Mask" "F.Paste")
-			(roundrect_rratio 0.09434)
+			(at -0.35 0 270)
+			(size 0.4 0.7)
+			(layers "F.Cu" "F.Mask")
+			(roundrect_rratio 0.125)
 			(net 4 "GND")
 			(pinfunction "K")
 			(pintype "passive")
+			(solder_paste_margin -0.05)
 		)
 		(pad "2" smd roundrect
-			(at 3.275 0 270)
-			(size 2.65 5.15)
-			(layers "F.Cu" "F.Mask" "F.Paste")
-			(roundrect_rratio 0.09434)
+			(at 0.35 0 270)
+			(size 0.4 0.7)
+			(layers "F.Cu" "F.Mask")
+			(roundrect_rratio 0.125)
 			(net 5 "SW")
 			(pinfunction "A")
 			(pintype "passive")
+			(solder_paste_margin -0.05)
 		)
 		(embedded_fonts no)
-		(model "${KICAD9_3DMODEL_DIR}/Diode_SMD.3dshapes/D_3220_8050Metric.wrl"
+		(model "${KICAD9_3DMODEL_DIR}/Diode_SMD.3dshapes/D_SOD-882.wrl"
 			(offset
 				(xyz 0 0 0)
@@
 	)
 	(segment
-		(start 116.815 96.76)
-		(end 123.18 96.76)
-		(width 0.2)
-		(layer "F.Cu")
-		(net 5)
-	)
-	(segment
 		(start 100.6 94.45)
 		(end 100.76 94.29)
@@
 	)
 	(segment
+		(start 116.815 96.76)
+		(end 118.8925 96.76)
+		(width 0.2)
+		(layer "F.Cu")
+		(net 5)
+	)
+	(segment
 		(start 100.6 98.296351)
 		(end 100.6 94.45)
 		(width 0.2)
 		(layer "F.Cu")
+		(net 5)
+	)
+	(segment
+		(start 118.8925 96.76)
+		(end 118.93 96.7225)
+		(width 0.2)
+		(layer "F.Cu")
