File: PCB/time-o-matic.kicad_sch (KiCad schematic)
At the start: 23 parts, among them J2 USB_C_Receptacle_USB2.0_14P, J5 Display Connector, U1 ESP32-WROOM-E, U2 MP1584EN-LF-P, U4 CH340C

Commit message: W
Parts:
- D1: footprint Diode_SMD:D_3220_8050Metric_Pad2.65x5.15mm_HandSolder -> Diode_SMD:D_SOD-882
Changed lines of the file:
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@@
 			)
 		)
-		(property "Footprint" "Diode_SMD:D_3220_8050Metric_Pad2.65x5.15mm_HandSolder"
+		(property "Footprint" "Diode_SMD:D_SOD-882"
 			(at 300.99 54.61 0)
 			(effects
